Commit message: .

File: xacro/gummi_description_ee.urdf.xacro (robot description, xacro)
@@ -23,19 +23,19 @@
       <geometry>
         <mesh
-          filename="package://gummi_ee_$(env ROS_GUMMI_EE)/meshes/lowerarm_preroll_d.STL" />
-      </geometry>
-      <material
-        name="">
-        <color
-          rgba="0.792156862745098 0.819607843137255 0.933333333333333 1" />
-      </material>
-    </visual>
-    <collision>
-      <origin
-        xyz="0 0 0"
-        rpy="0 0 0" />
-      <geometry>
-        <mesh
-          filename="package://gummi_ee_$(env ROS_GUMMI_EE)/meshes/lowerarm_preroll_d.STL" />
+          filename="package://gummi_rightee_$(env ROS_GUMMI_RIGHTEE)/meshes/lowerarm_preroll_d.STL" />
+      </geometry>
+      <material
+        name="">
+        <color
+          rgba="0.792156862745098 0.819607843137255 0.933333333333333 1" />
+      </material>
+    </visual>
+    <collision>
+      <origin
+        xyz="0 0 0"
+        rpy="0 0 0" />
+      <geometry>
+        <mesh
+          filename="package://gummi_rightee_$(env ROS_GUMMI_RIGHTEE)/meshes/lowerarm_preroll_d.STL" />
       </geometry>
     </collision>
@@ -76,19 +76,19 @@
       <geometry>
         <mesh
-          filename="package://gummi_ee_$(env ROS_GUMMI_EE)/meshes/lowerarm.STL" />
-      </geometry>
-      <material
-        name="">
-        <color
-          rgba="0.792156862745098 0.819607843137255 0.933333333333333 1" />
-      </material>
-    </visual>
-    <collision>
-      <origin
-        xyz="0 0 0"
-        rpy="0 0 0" />
-      <geometry>
-        <mesh
-          filename="package://gummi_ee_$(env ROS_GUMMI_EE)/meshes/lowerarm.STL" />
+          filename="package://gummi_rightee_$(env ROS_GUMMI_RIGHTEE)/meshes/lowerarm.STL" />
+      </geometry>
+      <material
+        name="">
+        <color
+          rgba="0.792156862745098 0.819607843137255 0.933333333333333 1" />
+      </material>
+    </visual>
+    <collision>
+      <origin
+        xyz="0 0 0"
+        rpy="0 0 0" />
+      <geometry>
+        <mesh
+          filename="package://gummi_rightee_$(env ROS_GUMMI_RIGHTEE)/meshes/lowerarm.STL" />
       </geometry>
     </collision>
@@ -132,19 +132,19 @@
       <geometry>
         <mesh
-          filename="package://gummi_ee_$(env ROS_GUMMI_EE)/meshes/wrist.STL" />
-      </geometry>
-      <material
-        name="">
-        <color
-          rgba="0.792156862745098 0.819607843137255 0.933333333333333 1" />
-      </material>
-    </visual>
-    <collision>
-      <origin
-        xyz="0 0 0"
-        rpy="0 0 0" />
-      <geometry>
-        <mesh
-          filename="package://gummi_ee_$(env ROS_GUMMI_EE)/meshes/wrist.STL" />
+          filename="package://gummi_rightee_$(env ROS_GUMMI_RIGHTEE)/meshes/wrist.STL" />
+      </geometry>
+      <material
+        name="">
+        <color
+          rgba="0.792156862745098 0.819607843137255 0.933333333333333 1" />
+      </material>
+    </visual>
+    <collision>
+      <origin
+        xyz="0 0 0"
+        rpy="0 0 0" />
+      <geometry>
+        <mesh
+          filename="package://gummi_rightee_$(env ROS_GUMMI_RIGHTEE)/meshes/wrist.STL" />
       </geometry>
     </collision>
@@ -203,19 +203,19 @@
       <geometry>
         <mesh
-          filename="package://gummi_ee_$(env ROS_GUMMI_EE)/meshes/i1.STL" />
-      </geometry>
-      <material
-        name="">
-        <color
-          rgba="0.792156862745098 0.819607843137255 0.933333333333333 1" />
-      </material>
-    </visual>
-    <collision>
-      <origin
-        xyz="0 0 0"
-        rpy="0 0 0" />
-      <geometry>
-        <mesh
-          filename="package://gummi_ee_$(env ROS_GUMMI_EE)/meshes/i1.STL" />
+          filename="package://gummi_rightee_$(env ROS_GUMMI_RIGHTEE)/meshes/i1.STL" />
+      </geometry>
+      <material
+        name="">
+        <color
+          rgba="0.792156862745098 0.819607843137255 0.933333333333333 1" />
+      </material>
+    </visual>
+    <collision>
+      <origin
+        xyz="0 0 0"
+        rpy="0 0 0" />
+      <geometry>
+        <mesh
+          filename="package://gummi_rightee_$(env ROS_GUMMI_RIGHTEE)/meshes/i1.STL" />
       </geometry>
     </collision>
@@ -262,19 +262,19 @@
       <geometry>
         <mesh
-          filename="package://gummi_ee_$(env ROS_GUMMI_EE)/meshes/i2.STL" />
-      </geometry>
-      <material
-        name="">
-        <color
-          rgba="0.792156862745098 0.819607843137255 0.933333333333333 1" />
-      </material>
-    </visual>
-    <collision>
-      <origin
-        xyz="0 0 0"
-        rpy="0 0 0" />
-      <geometry>
-        <mesh
-          filename="package://gummi_ee_$(env ROS_GUMMI_EE)/meshes/i2.STL" />
+          filename="package://gummi_rightee_$(env ROS_GUMMI_RIGHTEE)/meshes/i2.STL" />
+      </geometry>
+      <material
+        name="">
+        <color
+          rgba="0.792156862745098 0.819607843137255 0.933333333333333 1" />
+      </material>
+    </visual>
+    <collision>
+      <origin
+        xyz="0 0 0"
+        rpy="0 0 0" />
+      <geometry>
+        <mesh
+          filename="package://gummi_rightee_$(env ROS_GUMMI_RIGHTEE)/meshes/i2.STL" />
       </geometry>
     </collision>
@@ -321,19 +321,19 @@
       <geometry>
         <mesh
-          filename="package://gummi_ee_$(env ROS_GUMMI_EE)/meshes/i3.STL" />
-      </geometry>
-      <material
-        name="">
-        <color
-          rgba="0.792156862745098 0.819607843137255 0.933333333333333 1" />
-      </material>
-    </visual>
-    <collision>
-      <origin
-        xyz="0 0 0"
-        rpy="0 0 0" />
-      <geometry>
-        <mesh
-          filename="package://gummi_ee_$(env ROS_GUMMI_EE)/meshes/i3.STL" />
+          filename="package://gummi_rightee_$(env ROS_GUMMI_RIGHTEE)/meshes/i3.STL" />
+      </geometry>
+      <material
+        name="">
+        <color
+          rgba="0.792156862745098 0.819607843137255 0.933333333333333 1" />
+      </material>
+    </visual>
+    <collision>
+      <origin
+        xyz="0 0 0"
+        rpy="0 0 0" />
+      <geometry>
+        <mesh
+          filename="package://gummi_rightee_$(env ROS_GUMMI_RIGHTEE)/meshes/i3.STL" />
       </geometry>
     </collision>
@@ -380,19 +380,19 @@
       <geometry>
         <mesh
-          filename="package://gummi_ee_$(env ROS_GUMMI_EE)/meshes/i4.STL" />
-      </geometry>
-      <material
-        name="">
-        <color
-          rgba="0.792156862745098 0.819607843137255 0.933333333333333 1" />
-      </material>
-    </visual>
-    <collision>
-      <origin
-        xyz="0 0 0"
-        rpy="0 0 0" />
-      <geometry>
-        <mesh
-          filename="package://gummi_ee_$(env ROS_GUMMI_EE)/meshes/i4.STL" />
+          filename="package://gummi_rightee_$(env ROS_GUMMI_RIGHTEE)/meshes/i4.STL" />
+      </geometry>
+      <material
+        name="">
+        <color
+          rgba="0.792156862745098 0.819607843137255 0.933333333333333 1" />
+      </material>
+    </visual>
+    <collision>
+      <origin
+        xyz="0 0 0"
+        rpy="0 0 0" />
+      <geometry>
+        <mesh
+          filename="package://gummi_rightee_$(env ROS_GUMMI_RIGHTEE)/meshes/i4.STL" />
       </geometry>
     </collision>
@@ -439,19 +439,19 @@
       <geometry>
         <mesh
-          filename="package://gummi_ee_$(env ROS_GUMMI_EE)/meshes/i5.STL" />
-      </geometry>
-      <material
-        name="">
-        <color
-          rgba="0.792156862745098 0.819607843137255 0.933333333333333 1" />
-      </material>
-    </visual>
-    <collision>
-      <origin
-        xyz="0 0 0"
-        rpy="0 0 0" />
-      <geometry>
-        <mesh
-          filename="package://gummi_ee_$(env ROS_GUMMI_EE)/meshes/i5.STL" />
+          filename="package://gummi_rightee_$(env ROS_GUMMI_RIGHTEE)/meshes/i5.STL" />
+      </geometry>
+      <material
+        name="">
+        <color
+          rgba="0.792156862745098 0.819607843137255 0.933333333333333 1" />
+      </material>
+    </visual>
+    <collision>
+      <origin
+        xyz="0 0 0"
+        rpy="0 0 0" />
+      <geometry>
+        <mesh
+          filename="package://gummi_rightee_$(env ROS_GUMMI_RIGHTEE)/meshes/i5.STL" />
       </geometry>
     </collision>

Commit message: make it right

File: xacro/gummi_description_ee.urdf.xacro (robot description, xacro)
@@ -2,5 +2,5 @@
 <robot>
   <link
-    name="lowerarm_preroll_d">
+    name="right/lowerarm_preroll_d">
     <inertial>
       <origin
@@ -42,5 +42,5 @@
   </link>
   <joint
-    name="fastswitch"
+    name="right/fastswitch"
     type="fixed">
     <origin
@@ -48,12 +48,12 @@
       rpy="0 0 0" />
     <parent
-      link="lowerarm_preroll_u" />
-    <child
-      link="lowerarm_preroll_d" />
+      link="right/lowerarm_preroll_u" />
+    <child
+      link="right/lowerarm_preroll_d" />
     <axis
       xyz="0 0 0" />
   </joint>
   <link
-    name="lowerarm">
+    name="right/lowerarm">
     <inertial>
       <origin
@@ -95,5 +95,5 @@
   </link>
   <joint
-    name="forearm_roll"
+    name="right/forearm_roll"
     type="continuous">
     <origin
@@ -101,7 +101,7 @@
       rpy="0 0 0" />
     <parent
-      link="lowerarm_preroll_d" />
-    <child
-      link="lowerarm" />
+      link="right/lowerarm_preroll_d" />
+    <child
+      link="right/lowerarm" />
     <axis
       xyz="-1 0 0" />
@@ -111,5 +111,5 @@
   </joint>
   <link
-    name="wrist">
+    name="right/wrist">
     <inertial>
       <origin
@@ -151,5 +151,5 @@
   </link>
   <joint
-    name="wrist_pitch"
+    name="right/wrist_pitch"
     type="revolute">
     <origin
@@ -157,7 +157,7 @@
       rpy="0 0 0" />
     <parent
-      link="lowerarm" />
-    <child
-      link="wrist" />
+      link="right/lowerarm" />
+    <child
+      link="right/wrist" />
     <axis
       xyz="0 1 0" />
@@ -173,14 +173,14 @@
   offset and a multiplication rate. check ros docs for details
   -->
-  <joint name="gripper" type="revolute">
+  <joint name="right/gripper" type="revolute">
     <origin rpy="0 0 0" xyz="0 0 0"/>
-    <parent link="wrist"/>
-    <child link="dummygripper"/>
+    <parent link="right/wrist"/>
+    <child link="right/dummygripper"/>
     <axis xyz="0 1 0"/>
     <limit effort="0" lower="0" upper="2" velocity="0"/>
   </joint>
-  <link name="dummygripper"/>
-  <link
-    name="i1">
+  <link name="right/dummygripper"/>
+  <link
+    name="right/i1">
     <inertial>
       <origin
@@ -222,5 +222,5 @@
   </link>
   <joint
-    name="i1f"
+    name="right/i1f"
     type="revolute">
     <origin
@@ -228,7 +228,7 @@
       rpy="-0.79367 0.12795 -0.91441" />
     <parent
-      link="wrist" />
-    <child
-      link="i1" />
+      link="right/wrist" />
+    <child
+      link="right/i1" />
     <axis
       xyz="0 -1 0" />
@@ -238,8 +238,8 @@
       effort="0"
       velocity="0" />
-    <mimic joint="gripper"/>
-  </joint>
-  <link
-    name="i2">
+    <mimic joint="right/gripper"/>
+  </joint>
+  <link
+    name="right/i2">
     <inertial>
       <origin
@@ -281,5 +281,5 @@
   </link>
   <joint
-    name="i2f"
+    name="right/i2f"
     type="revolute">
     <origin
@@ -287,7 +287,7 @@
       rpy="-6.9389E-16 -8.4436E-17 -0.12109" />
     <parent
-      link="wrist" />
-    <child
-      link="i2" />
+      link="right/wrist" />
+    <child
+      link="right/i2" />
     <axis
       xyz="0 -1 0" />
@@ -297,8 +297,8 @@
       effort="0"
       velocity="0" />
-    <mimic joint="gripper"/>
-  </joint>
-  <link
-    name="i3">
+    <mimic joint="right/gripper"/>
+  </joint>
+  <link
+    name="right/i3">
     <inertial>
       <origin
@@ -340,5 +340,5 @@
   </link>
   <joint
-    name="i3f"
+    name="right/i3f"
     type="revolute">
     <origin
@@ -346,7 +346,7 @@
       rpy="-1.0408E-15 -5.7778E-30 -5.5511E-15" />
     <parent
-      link="wrist" />
-    <child
-      link="i3" />
+      link="right/wrist" />
+    <child
+      link="right/i3" />
     <axis
       xyz="0 -1 0" />
@@ -356,8 +356,8 @@
       effort="0"
       velocity="0" />
-    <mimic joint="gripper"/>
-  </joint>
-  <link
-    name="i4">
+    <mimic joint="right/gripper"/>
+  </joint>
+  <link
+    name="right/i4">
     <inertial>
       <origin
@@ -399,5 +399,5 @@
   </link>
   <joint
-    name="i4f"
+    name="right/i4f"
     type="revolute">
     <origin
@@ -405,7 +405,7 @@
       rpy="-1.0408E-15 1.4051E-16 0.13418" />
     <parent
-      link="wrist" />
-    <child
-      link="i4" />
+      link="right/wrist" />
+    <child
+      link="right/i4" />
     <axis
       xyz="0 -1 0" />
@@ -415,8 +415,8 @@
       effort="0"
       velocity="0" />
-    <mimic joint="gripper"/>
-  </joint>
-  <link
-    name="i5">
+    <mimic joint="right/gripper"/>
+  </joint>
+  <link
+    name="right/i5">
     <inertial>
       <origin
@@ -458,5 +458,5 @@
   </link>
   <joint
-    name="i5f"
+    name="right/i5f"
     type="revolute">
     <origin
@@ -464,7 +464,7 @@
       rpy="1.9429E-14 -3.8109E-15 0.19369" />
     <parent
-      link="wrist" />
-    <child
-      link="i5" />
+      link="right/wrist" />
+    <child
+      link="right/i5" />
     <axis
       xyz="0 -1 0" />
@@ -474,5 +474,5 @@
       effort="0"
       velocity="0" />
-    <mimic joint="gripper"/>
+    <mimic joint="right/gripper"/>
   </joint>
 </robot>

File: xacro/gummi_ee.srdf.xacro (robot description, xacro)
@@ -2,47 +2,47 @@
 <robot name="gummi" xmlns:xacro="http://www.ros.org/wiki/xacro">
 <xacro:macro name="group_right_arm_ee">
-    <joint name="forearm_roll" />
-    <joint name="wrist_pitch" />
+    <joint name="right/forearm_roll" />
+    <joint name="right/wrist_pitch" />
 </xacro:macro>
 <xacro:macro name="group_right_gripper_ee">
   <group name="right_gripper">
-    <link name="wrist"/>
-    <joint name="gripper"/>
+    <link name="right/wrist"/>
+    <joint name="right/gripper"/>
   </group>
 </xacro:macro>
 <xacro:macro name="group_state_right_arm_ee">
-  <joint name="forearm_roll" value="0" />
-  <joint name="wrist_pitch" value="0" />
+  <joint name="right/forearm_roll" value="0" />
+  <joint name="right/wrist_pitch" value="0" />
 </xacro:macro>
 <xacro:macro name="end_effector_ee">
   <!--END EFFECTOR: Purpose: Represent information about an end effector.-->
-<end_effector group="right_gripper" name="right_eef" parent_link="wrist" parent_group="right_arm"/>
+<end_effector group="right_gripper" name="right_eef" parent_link="right/wrist" parent_group="right_arm"/>
 </xacro:macro>
 <xacro:macro name="disable_collisions_ee">
-  <!-- <disable_collisions link1="right_hand" link2="wrist" reason="Never" />
-  <disable_collisions link1="right_hand" link2="gripper_link" reason="Never" /> -->
-  <disable_collisions link1="i1" link2="lowerarm" reason="Never" />
-  <disable_collisions link1="i2" link2="lowerarm" reason="Never" />
-  <disable_collisions link1="i3" link2="lowerarm" reason="Never" />
-  <disable_collisions link1="i4" link2="lowerarm" reason="Never" />
-  <disable_collisions link1="i5" link2="lowerarm" reason="Never" />
-  <disable_collisions link1="i1" link2="wrist" reason="Never" />
-  <disable_collisions link1="i2" link2="wrist" reason="Never" />
-  <disable_collisions link1="i3" link2="wrist" reason="Never" />
-  <disable_collisions link1="i4" link2="wrist" reason="Never" />
-  <disable_collisions link1="i5" link2="wrist" reason="Never" />
-  <disable_collisions link1="i1" link2="i2" reason="Never" />
-  <disable_collisions link1="i1" link2="i3" reason="Never" />
-  <disable_collisions link1="i1" link2="i4" reason="Never" />
-  <disable_collisions link1="i1" link2="i5" reason="Never" />
-  <disable_collisions link1="i2" link2="i3" reason="Never" />
-  <disable_collisions link1="i2" link2="i4" reason="Never" />
-  <disable_collisions link1="i2" link2="i5" reason="Never" />
-  <disable_collisions link1="i3" link2="i4" reason="Never" />
-  <disable_collisions link1="i3" link2="i5" reason="Never" />
-  <disable_collisions link1="i4" link2="i5" reason="Never" />
-  <disable_collisions link1="lowerarm" link2="lowerarm_preroll_d" reason="Adjacent" />
-  <disable_collisions link1="lowerarm" link2="wrist" reason="Adjacent" />
-  <disable_collisions link1="lowerarm_preroll_d" link2="wrist" reason="Never" />
+  <!-- <disable_collisions link1="right/right_hand" link2="right/wrist" reason="Never" />
+  <disable_collisions link1="right/right_hand" link2="right/gripper_link" reason="Never" /> -->
+  <disable_collisions link1="right/i1" link2="right/lowerarm" reason="Never" />
+  <disable_collisions link1="right/i2" link2="right/lowerarm" reason="Never" />
+  <disable_collisions link1="right/i3" link2="right/lowerarm" reason="Never" />
+  <disable_collisions link1="right/i4" link2="right/lowerarm" reason="Never" />
+  <disable_collisions link1="right/i5" link2="right/lowerarm" reason="Never" />
+  <disable_collisions link1="right/i1" link2="right/wrist" reason="Never" />
+  <disable_collisions link1="right/i2" link2="right/wrist" reason="Never" />
+  <disable_collisions link1="right/i3" link2="right/wrist" reason="Never" />
+  <disable_collisions link1="right/i4" link2="right/wrist" reason="Never" />
+  <disable_collisions link1="right/i5" link2="right/wrist" reason="Never" />
+  <disable_collisions link1="right/i1" link2="right/i2" reason="Never" />
+  <disable_collisions link1="right/i1" link2="right/i3" reason="Never" />
+  <disable_collisions link1="right/i1" link2="right/i4" reason="Never" />
+  <disable_collisions link1="right/i1" link2="right/i5" reason="Never" />
+  <disable_collisions link1="right/i2" link2="right/i3" reason="Never" />
+  <disable_collisions link1="right/i2" link2="right/i4" reason="Never" />
+  <disable_collisions link1="right/i2" link2="right/i5" reason="Never" />
+  <disable_collisions link1="right/i3" link2="right/i4" reason="Never" />
+  <disable_collisions link1="right/i3" link2="right/i5" reason="Never" />
+  <disable_collisions link1="right/i4" link2="right/i5" reason="Never" />
+  <disable_collisions link1="right/lowerarm" link2="right/lowerarm_preroll_d" reason="Adjacent" />
+  <disable_collisions link1="right/lowerarm" link2="right/wrist" reason="Adjacent" />
+  <disable_collisions link1="right/lowerarm_preroll_d" link2="right/wrist" reason="Never" />
 </xacro:macro>
 </robot>
